File: board/fluxgate.kicad_pcb (KiCad board)
At the start: 2 copper layers, 45.1 x 86.6 mm, 59 parts, among them J1 Drive coil, J2 Drive coil, J3 5 V, J5 Prog, J7 Micro_SD_Card, J8 Sense, J9 Sense, Q1 2N7000, Q3 2N3906, Q4 2N7000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

Commit message: Start working on measurement
Parts:
- C13: value 10 nF -> 100 nF
- R10: value 5k -> 5k7
- R13: value 50 -> 57
- R16: value 21k -> 22k
- R6: value 500 -> 1k
- R9: value 50 -> 47
- Y1: value Crystal -> 32.768 kHz
Connections:
- U1 pad 1: unconnected-(U1-PA3-Pad1) -> ADC+
- U1 pad 31: ADC+ -> unconnected-(U1-PA1-Pad31)
Routing:
- net ADC+: track 76.4 -> 78.6 mm, vias 0 -> 2
Changed lines of the file:
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@@
 	(net 35 "unconnected-(U1-PF5-Pad25)")
 	(net 36 "unconnected-(U1-PD4-Pad14)")
-	(net 37 "unconnected-(U1-PA3-Pad1)")
+	(net 37 "unconnected-(U1-PA1-Pad31)")
 	(net 38 "unconnected-(U1-PF4-Pad24)")
 	(net 39 "unconnected-(U1-PF3-Pad23)")
@@
 			(size 1.6 0.55)
 			(layers "F.Cu" "F.Paste" "F.Mask")
-			(net 37 "unconnected-(U1-PA3-Pad1)")
+			(net 10 "ADC+")
 			(pinfunction "PA3")
 			(pintype "bidirectional")
@@
 			(size 1.6 0.55)
 			(layers "F.Cu" "F.Paste" "F.Mask")
-			(net 10 "ADC+")
+			(net 37 "unconnected-(U1-PA1-Pad31)")
 			(pinfunction "PA1")
 			(pintype "bidirectional")
@@
 			)
 		)
-		(property "Value" "5k"
+		(property "Value" "5k7"
 			(at 5.08 2.37 0)
 			(layer "F.Fab")
@@
 			)
 		)
-		(property "Value" "10 nF"
+		(property "Value" "100 nF"
 			(at 1.25 2.3 0)
 			(layer "F.Fab")
@@
 			)
 		)
-		(property "Value" "Crystal"
+		(property "Value" "32.768 kHz"
 			(at 1.9 2.85 0)
 			(layer "F.Fab")
@@
 			)
 		)
-		(property "Value" "21k"
+		(property "Value" "22k"
 			(at 5.08 2.37 0)
 			(layer "F.Fab")
@@
 			)
 		)
-		(property "Value" "50"
+		(property "Value" "57"
 			(at 5.08 2.37 0)
 			(layer "F.Fab")
@@
 			)
 		)
-		(property "Value" "50"
+		(property "Value" "47"
 			(at 5.08 2.37 0)
 			(layer "F.Fab")
@@
 			)
 		)
-		(property "Value" "500"
+		(property "Value" "1k"
 			(at 5.08 2.37 0)
 			(layer "F.Fab")
@@
 	)
 	(segment
+		(start 166.157169 63.287169)
+		(end 166.157169 63.331831)
+		(width 0.5)
+		(layer "F.Cu")
+		(net 10)
+	)
+	(segment
 		(start 178.205001 102.083999)
 		(end 178.205001 98.019999)
@@
 	)
 	(segment
-		(start 172.72 69.85)
-		(end 165.195 62.325)
-		(width 0.5)
-		(layer "F.Cu")
-		(net 10)
-	)
-	(segment
 		(start 179.705 93.218)
 		(end 179.578 93.091)
@@
 	)
 	(segment
+		(start 165.989 63.119)
+		(end 166.157169 63.287169)
+		(width 0.5)
+		(layer "F.Cu")
+		(net 10)
+	)
+	(segment
+		(start 167.386 61.976)
+		(end 167.386 59.939)
+		(width 0.5)
+		(layer "F.Cu")
+		(net 10)
+	)
+	(segment
 		(start 167.62 104.755)
 		(end 172.065 104.755)
@@
 	)
 	(segment
+		(start 167.386 59.939)
+		(end 167.445 59.88)
+		(width 0.5)
+		(layer "F.Cu")
+		(net 10)
+	)
+	(segment
 		(start 167.112 104.247)
 		(end 167.62 104.755)
@@
 	)
 	(segment
-		(start 174.879 105.41)
-		(end 178.205001 102.083999)
+		(start 172.72 69.85)
+		(end 165.989 63.119)
 		(width 0.5)
 		(layer "F.Cu")
@@
 	)
 	(segment
-		(start 165.195 62.325)
-		(end 165.195 61.33)
+		(start 174.879 105.41)
+		(end 178.205001 102.083999)
 		(width 0.5)
 		(layer "F.Cu")
@@
 		(net 10)
 	)
+	(via
+		(at 166.157169 63.331831)
+		(size 0.6)
+		(drill 0.3)
+		(layers "F.Cu" "B.Cu")
+		(net 10)
+	)
+	(via
+		(at 167.386 61.976)
+		(size 0.6)
+		(drill 0.3)
+		(layers "F.Cu" "B.Cu")
+		(net 10)
+	)
+	(segment
+		(start 167.386 62.103)
+		(end 167.386 61.976)
+		(width 0.5)
+		(layer "B.Cu")
+		(net 10)
+	)
+	(segment
+		(start 166.157169 63.331831)
+		(end 167.386 62.103)
+		(width 0.5)
+		(layer "B.Cu")
+		(net 10)
+	)
